Commit message: rename camera models to sensor models

File: humanoid/ARX/arx_lift_description/urdf/arx_lift.urdf (robot description, URDF)
Before this commit: robot arx_lift, 37 links, 36 joints
Links:
- link left_camera: geometry visual mesh filename=package://sensor_models/meshes/d405/d405.obj
- link right_camera: geometry visual mesh filename=package://sensor_models/meshes/d405/d405.obj

File: humanoid/ARX/arx_lift_description/urdf/arx_lift_r5.urdf (robot description, URDF)
Before this commit: robot arx_lift, 37 links, 36 joints
Links:
- link left_camera: geometry visual mesh filename=package://sensor_models/meshes/d405/d405.obj
- link right_camera: geometry visual mesh filename=package://sensor_models/meshes/d405/d405.obj

File: humanoid/ARX/x7s_description/urdf/x7s.urdf (robot description, URDF)
Before this commit: robot X7S, 26 links, 25 joints
Links:
- link head_camera: geometry visual mesh filename=package://sensor_models/meshes/d405/d405.obj

File: humanoid/ARX/x7s_description/xacro/x7s.xacro (robot description, xacro)
@@ -149,5 +149,5 @@
       <visual>
         <geometry>
-          <mesh filename="file://$(find camera_models)/meshes/d405/d405.obj"/>
+          <mesh filename="file://$(find sensor_models)/meshes/d405/d405.obj"/>
         </geometry>
       </visual>

File: humanoid/Agibot/agibot_g1_description/xacro/120s_camera_stand.xacro (robot description, xacro)
@@ -22,5 +22,5 @@
 			<visual>
 				<geometry>
-					<mesh filename="file://$(find camera_models)/meshes/d405/d405.obj"/>
+					<mesh filename="file://$(find sensor_models)/meshes/d405/d405.obj"/>
 				</geometry>
 			</visual>

File: humanoid/Agibot/agibot_g1_description/xacro/omnipicker_camera_stand.xacro (robot description, xacro)
@@ -23,5 +23,5 @@
 			<visual>
 				<geometry>
-					<mesh filename="file://$(find camera_models)/meshes/d405/d405.obj"/>
+					<mesh filename="file://$(find sensor_models)/meshes/d405/d405.obj"/>
 				</geometry>
 			</visual>

File: humanoid/Galaxea/galaxea_r1_description/urdf/galaxea_r1.urdf (robot description, URDF)
Before this commit: robot R1, 36 links, 35 joints
Links:
- link left_realsense_link: geometry collision mesh filename=package://galaxea_r1_description/meshes/camera_stand.obj; visual mesh filename=package://galaxea_r1_description/meshes/camera_stand.obj
- link right_realsense_link: geometry collision mesh filename=package://galaxea_r1_description/meshes/camera_stand.obj; visual mesh filename=package://galaxea_r1_description/meshes/camera_stand.obj

File: humanoid/Galaxea/galaxea_r1_description/xacro/realsense.xacro (robot description, xacro)
@@ -19,5 +19,5 @@
         <origin rpy="${PI/2} ${-PI/2} 0" xyz="0.0325 0 0"/>
         <geometry>
-          <mesh filename="file://$(find camera_models)/meshes/d435/d435.obj"/>
+          <mesh filename="file://$(find sensor_models)/meshes/d435/d435.obj"/>
         </geometry>
       </visual>

File: humanoid/Galaxea/galaxea_r1pro_description/urdf/galaxea_r1pro.urdf (robot description, URDF)
Before this commit: robot R1Pro, 38 links, 37 joints
Links:
- link left_realsense_link: geometry collision mesh filename=package://galaxea_r1_description/meshes/camera_stand.obj; visual mesh filename=package://galaxea_r1_description/meshes/camera_stand.obj
- link right_realsense_link: geometry collision mesh filename=package://galaxea_r1_description/meshes/camera_stand.obj; visual mesh filename=package://galaxea_r1_description/meshes/camera_stand.obj

File: humanoid/Galaxea/galaxea_r1pro_description/xacro/realsense.xacro (robot description, xacro)
@@ -19,5 +19,5 @@
         <origin rpy="${PI/2} ${-PI/2} 0" xyz="0.0325 0 0"/>
         <geometry>
-          <mesh filename="file://$(find camera_models)/meshes/d435/d435.obj"/>
+          <mesh filename="file://$(find sensor_models)/meshes/d435/d435.obj"/>
         </geometry>
       </visual>

File: manipulator/ARX/arx5_description/urdf/arx5.urdf (robot description, URDF)
Before this commit: robot ARX 5, 14 links, 13 joints
Links:
- link camera: geometry visual mesh filename=package://sensor_models/meshes/d405/d405.obj

File: manipulator/ARX/arx5_description/urdf/arx5_agilex.urdf (robot description, URDF)
Before this commit: robot ARX 5, 14 links, 13 joints
Links:
- link camera: geometry visual mesh filename=package://sensor_models/meshes/d405/d405.obj

File: manipulator/ARX/arx5_description/urdf/arx5_r5.urdf (robot description, URDF)
Before this commit: robot ARX 5, 14 links, 13 joints
Links:
- link camera: geometry visual mesh filename=package://sensor_models/meshes/d405/d405.obj

File: manipulator/ARX/arx5_description/xacro/R5.xacro (robot description, xacro)
@@ -311,5 +311,5 @@
 				<visual>
 					<geometry>
-						<mesh filename="file://$(find camera_models)/meshes/d405/d405.obj"/>
+						<mesh filename="file://$(find sensor_models)/meshes/d405/d405.obj"/>
 					</geometry>
 				</visual>
@@ -337,5 +337,5 @@
 				<visual>
 					<geometry>
-						<mesh filename="file://$(find camera_models)/meshes/d435/d435.obj"/>
+						<mesh filename="file://$(find sensor_models)/meshes/d435/d435.obj"/>
 					</geometry>
 				</visual>

File: manipulator/ARX/arx5_description/xacro/X5.xacro (robot description, xacro)
@@ -302,5 +302,5 @@
         <visual>
           <geometry>
-            <mesh filename="file://$(find camera_models)/meshes/d405/d405.obj"/>
+            <mesh filename="file://$(find sensor_models)/meshes/d405/d405.obj"/>
           </geometry>
         </visual>
@@ -328,5 +328,5 @@
         <visual>
           <geometry>
-            <mesh filename="file://$(find camera_models)/meshes/d435/d435.obj"/>
+            <mesh filename="file://$(find sensor_models)/meshes/d435/d435.obj"/>
           </geometry>
         </visual>

File: manipulator/AgileX/agilex_aloha_description/urdf/agilex_aloha_v1.urdf (robot description, URDF)
Before this commit: robot AgileX Aloha, 46 links, 45 joints
Links:
- link camera_link1: geometry visual mesh filename=package://agilex_aloha_description/meshes/aloha_v1/camera_s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; visual mesh filename=package://sensor_models/meshes/d435/d435.obj
- link camera_link2: geometry visual mesh filename=package://agilex_aloha_description/meshes/aloha_v1/camera_s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; visual mesh filename=package://sensor_models/meshes/d435/d435.obj
- link left_camera: geometry visual mesh filename=package://sensor_models/meshes/d435/d435.obj
- link lidar_link: geometry visual mesh filename=package://sensor_models/meshes/mid360/mid360.obj
- link right_camera: geometry visual mesh filename=package://sensor_models/meshes/d435/d435.obj

File: manipulator/AgileX/agilex_aloha_description/urdf/agilex_aloha_v1_x5.urdf (robot description, URDF)
Before this commit: robot AgileX Aloha, 46 links, 45 joints
Links:
- link camera_link1: geometry visual mesh filename=package://agilex_aloha_description/meshes/aloha_v1/camera_s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; visual mesh filename=package://sensor_models/meshes/d435/d435.obj
- link camera_link2: geometry visual mesh filename=package://agilex_aloha_description/meshes/aloha_v1/camera_s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; visual mesh filename=package://sensor_models/meshes/d435/d435.obj
- link left_camera: geometry visual mesh filename=package://sensor_models/meshes/d435/d435.obj
- link lidar_link: geometry visual mesh filename=package://sensor_models/meshes/mid360/mid360.obj
- link right_camera: geometry visual mesh filename=package://sensor_models/meshes/d435/d435.obj

File: manipulator/AgileX/agilex_aloha_description/urdf/agilex_aloha_v2-1.urdf (robot description, URDF)
Before this commit: robot AgileX Aloha, 33 links, 32 joints
Links:
- link camera_link: geometry visual mesh filename=package://sensor_models/meshes/dabai/dabai.obj
- link lidar_link: geometry visual mesh filename=package://sensor_models/meshes/mid360/mid360.obj

File: manipulator/AgileX/agilex_aloha_description/urdf/agilex_aloha_v2.urdf (robot description, URDF)
Before this commit: robot AgileX Aloha, 38 links, 37 joints
Links:
- link camera_link: geometry visual mesh filename=package://sensor_models/meshes/dabai/dabai.obj
- link lidar_link: geometry visual mesh filename=package://sensor_models/meshes/mid360/mid360.obj

File: manipulator/AgileX/agilex_aloha_description/xacro/aloha_split.xacro (robot description, xacro)
@@ -44,5 +44,5 @@
     <visual>
       <geometry>
-        <mesh filename="file://$(find camera_models)/meshes/dabai/dabai.obj"/>
+        <mesh filename="file://$(find sensor_models)/meshes/dabai/dabai.obj"/>
       </geometry>
     </visual>
@@ -67,5 +67,5 @@
     <visual>
       <geometry>
-        <mesh filename="file://$(find camera_models)/meshes/mid360/mid360.obj"/>
+        <mesh filename="file://$(find sensor_models)/meshes/mid360/mid360.obj"/>
       </geometry>
     </visual>
@@ -120,5 +120,5 @@
     <visual>
       <geometry>
-        <mesh filename="file://$(find camera_models)/meshes/dabai/dabai.obj"/>
+        <mesh filename="file://$(find sensor_models)/meshes/dabai/dabai.obj"/>
       </geometry>
     </visual>
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