Commit message: agilex aloha component fix

File: humanoid/Agibot/agibot_g1_description/xacro/g1_base.xacro (robot description, xacro)
@@ -73,4 +73,9 @@
 					izz="0.0051541"/>
 		</inertial>
+		<visual>
+			<geometry>
+				<mesh filename="file://$(find agibot_g1_description)/meshes/base/wheel.obj" scale="1 1 1"/>
+			</geometry>
+		</visual>
 		<collision>
 			<origin rpy="1.5708 0 0"/>
@@ -110,4 +115,9 @@
 					izz="0.0051541"/>
 		</inertial>
+		<visual>
+			<geometry>
+				<mesh filename="file://$(find agibot_g1_description)/meshes/base/wheel.obj" scale="1 -1 1"/>
+			</geometry>
+		</visual>
 		<collision>
 			<origin rpy="1.5708 0 0"/>

File: manipulator/AgileX/agilex_aloha_description/xacro/aloha_v1.xacro (robot description, xacro)
@@ -3,146 +3,5 @@
 	<xacro:macro name="aloha_v1" params="arm:=r5">
 		<xacro:include filename="$(find agilex_aloha_description)/xacro/base/tracer.xacro"/>
-		<link name="body_link">
-			<inertial>
-				<origin xyz="0.015107 -0.027922 0.00013672"/>
-				<mass value="3.736"/>
-				<inertia ixx="0.097545" ixy="-9.2609E-06" ixz="0.00015366" iyy="0.045841" iyz="-0.0020459" izz="0.084773"/>
-			</inertial>
-			<visual>
-				<geometry>
-					<mesh filename="file://$(find agilex_aloha_description)/meshes/aloha_v1/body_link.obj"/>
-				</geometry>
-			</visual>
-			<collision>
-				<geometry>
-					<mesh filename="file://$(find agilex_aloha_description)/meshes/aloha_v1/body_link.obj"/>
-				</geometry>
-			</collision>
-		</link>
-		<joint name="box2" type="fixed">
-			<origin xyz="0 0 0.15"/>
-			<parent link="base_footprint"/>
-			<child link="body_link"/>
-		</joint>
-		<link name="camera_base_link">
-			<inertial>
-				<origin xyz="-0.00862442289199344 -5.31672329634469E-08 0.170092831004467"/>
-				<mass value="0.336269569361489"/>
-				<inertia
-						ixx="0.00580628296841397"
-						ixy="3.98435937176716E-10"
-						ixz="-2.42350052877161E-05"
-						iyy="0.00582602200678083"
-						iyz="2.9180594404216E-10"
-						izz="0.000186894283496158"/>
-			</inertial>
-			<visual>
-				<geometry>
-					<mesh filename="file://$(find agilex_aloha_description)/meshes/aloha_v1/camera_support.obj"/>
-				</geometry>
-			</visual>
-			<collision>
-				<geometry>
-					<mesh filename="file://$(find agilex_aloha_description)/meshes/aloha_v1/camera_support.obj"/>
-				</geometry>
-			</collision>
-		</link>
-		<joint name="camera_to_box1" type="fixed">
-			<origin xyz="0.18 0 0.626"/>
-			<parent link="body_link"/>
-			<child link="camera_base_link"/>
-			<axis/>
-		</joint>
-		<link name="camera_link1">
-			<inertial>
-				<origin xyz="-0.0292387906463559 0.000126439620513119 -0.000724950892729725"/>
-				<mass value="0.0877001598245188"/>
-				<inertia
-						ixx="7.77343248794949E-05"
-						ixy="2.44922634558373E-07"
-						ixz="1.73341747661077E-08"
-						iyy="9.73521513961785E-06"
-						iyz="-2.86133018917868E-09"
-						izz="7.74948757118157E-05"/>
-			</inertial>
-			<visual>
-				<geometry>
-					<mesh filename="file://$(find agilex_aloha_description)/meshes/aloha_v1/camera_stand.obj"/>
-				</geometry>
-			</visual>
-			<visual>
-				<geometry>
-					<mesh filename="file://$(find sensor_models)/meshes/d435/d435.obj"/>
-				</geometry>
-			</visual>
-		</link>
-		<joint name="camera_joint1" type="fixed">
-			<origin xyz="0.071198 0 0.10384" rpy="0 0.26931 0"/>
-			<parent link="camera_base_link"/>
-			<child link="camera_link1"/>
-		</joint>
-		<link name="camera_link2">
-			<inertial>
-				<origin xyz="-0.0292307474530399 0.000126438461566014 -0.000753459207498031"/>
-				<mass value="0.0877001605148491"/>
-				<inertia
-						ixx="7.77338961798341E-05"
-						ixy="2.44922367048273E-07"
-						ixz="1.80373226250749E-08"
-						iyy="9.73521616927317E-06"
-						iyz="-2.86130173714525E-09"
-						izz="7.74953085203139E-05"/>
-			</inertial>
-			<visual>
-				<geometry>
-					<mesh filename="file://$(find agilex_aloha_description)/meshes/aloha_v1/camera_stand.obj"/>
-				</geometry>
-			</visual>
-			<visual>
-				<geometry>
-					<mesh filename="file://$(find sensor_models)/meshes/d435/d435.obj"/>
-				</geometry>
-			</visual>
-		</link>
-		<joint name="camera_joint2" type="fixed">
-			<origin xyz="-0.14 0 0.5" rpy="0 0.011358 0"/>
-			<parent link="camera_link1"/>
-			<child link="camera_link2"/>
-		</joint>
-		<link name="lidar_link">
-			<inertial>
-				<origin xyz="-0.0022133 -0.00090659 0.025996"/>
-				<mass value="0.048617"/>
-				<inertia
-						ixx="1.0358E-05"
-						ixy="9.2377E-09"
-						ixz="-2.6386E-07"
-						iyy="1.0387E-05"
-						iyz="-2.6377E-07"
-						izz="1.7919E-05"/>
-			</inertial>
-			<visual>
-				<geometry>
-					<mesh filename="file://$(find sensor_models)/meshes/mid360/mid360.obj"/>
-				</geometry>
-			</visual>
-		</link>
-		<joint name="lidar_joint" type="fixed">
-			<origin xyz="0.22937 0 0.040672"/>
-			<parent link="body_link"/>
-			<child link="lidar_link"/>
-		</joint>
-		<joint name="fl_base_joint" type="fixed">
-			<origin xyz="0.233 0.3 0.7775"/>
-			<parent link="base_footprint"/>
-			<child link="left_base_link"/>
-			<axis xyz="0.0 0.0 1.0"/>
-		</joint>
-		<joint name="fr_base_joint" type="fixed">
-			<origin xyz="0.233 -0.3 0.7775"/>
-			<parent link="base_footprint"/>
-			<child link="right_base_link"/>
-			<axis xyz="0.0 0.0 1.0"/>
-		</joint>
+		<xacro:include filename="$(find agilex_aloha_description)/xacro/body/v1.xacro"/>
 		<xacro:if value="${arm == 'x5'}">
 			<xacro:include filename="$(find arx5_description)/xacro/X5.xacro"/>

File: manipulator/AgileX/agilex_aloha_description/xacro/aloha_v2.xacro (robot description, xacro)
@@ -3,4 +3,5 @@
 	<xacro:macro name="aloha_v2" params="chassis:=tracer enable_master:=false">
 		<xacro:include filename="$(find piper_description)/xacro/Piper.xacro"/>
+		<xacro:include filename="$(find agilex_aloha_description)/xacro/body/v2.xacro"/>
 		<xacro:if value="${chassis == 'tracer'}">
 			<xacro:include filename="$(find agilex_aloha_description)/xacro/base/tracer.xacro"/>
@@ -9,90 +10,6 @@
 			<xacro:include filename="$(find agilex_aloha_description)/xacro/base/tracer_v2.xacro"/>
 		</xacro:if>
-		<!-- aloha base -->
-		<link name="body_Link">
-			<inertial>
-				<origin xyz="0.015107 -0.027922 0.00013672"/>
-				<mass value="3.736"/>
-				<inertia ixx="0.097545" ixy="-9.2609E-06" ixz="0.00015366" iyy="0.045841" iyz="-0.0020459" izz="0.084773"/>
-			</inertial>
-			<visual>
-				<geometry>
-					<mesh filename="file://$(find agilex_aloha_description)/meshes/aloha_v2/body.obj"/>
-				</geometry>
-			</visual>
-			<collision>
-				<geometry>
-					<mesh filename="file://$(find agilex_aloha_description)/meshes/aloha_v2/body.obj"/>
-				</geometry>
-			</collision>
-		</link>
-		<joint name="body_joint" type="fixed">
-			<origin xyz="0 0 0.168"/>
-			<parent link="base_footprint"/>
-			<child link="body_Link"/>
-			<axis/>
-		</joint>
-		<link name="camera_link">
-			<inertial>
-				<origin xyz="-0.011443 2.4833E-05 -0.0012615"/>
-				<mass value="0.020053"/>
-				<inertia
-						ixx="1.1181E-05"
-						ixy="1.204E-07"
-						ixz="4.9068E-08"
-						iyy="2.2587E-06"
-						iyz="5.7637E-07"
-						izz="1.0097E-05"/>
-			</inertial>
-			<visual>
-				<geometry>
-					<mesh filename="file://$(find sensor_models)/meshes/dabai/dabai.obj"/>
-				</geometry>
-			</visual>
-		</link>
-		<joint name="camera_joint" type="fixed">
-			<origin xyz="0.24007 0 0.91661" rpy="0 0.825 0"/>
-			<parent link="body_Link"/>
-			<child link="camera_link"/>
-		</joint>
-		<link name="lidar_link">
-			<inertial>
-				<origin xyz="-0.0022133 -0.00090659 0.025996"/>
-				<mass value="0.048617"/>
-				<inertia
-						ixx="1.0358E-05"
-						ixy="9.2377E-09"
-						ixz="-2.6386E-07"
-						iyy="1.0387E-05"
-						iyz="-2.6377E-07"
-						izz="1.7919E-05"/>
-			</inertial>
-			<visual>
-				<geometry>
-					<mesh filename="file://$(find sensor_models)/meshes/mid360/mid360.obj"/>
-				</geometry>
-			</visual>
-		</link>
-		<joint name="lidar_joint" type="fixed">
-			<origin xyz="0.27289 0 0.01488"/>
-			<parent link="body_Link"/>
-			<child link="lidar_link"/>
-		</joint>
-		<!--***************************** front-left ****************************** -->
 		<xacro:Piper name="left"/>
-		<joint name="left_base_joint" type="fixed">
-			<origin xyz="0.23875 0.3 0.607"/>
-			<parent link="body_Link"/>
-			<child link="left_base_link"/>
-			<axis xyz="0 0 1"/>
-		</joint>
-		<!--***************************** front-right ****************************** -->
 		<xacro:Piper name="right"/>
-		<joint name="right_base_joint" type="fixed">
-			<origin xyz="0.23875 -0.3 0.607"/>
-			<parent link="body_Link"/>
-			<child link="right_base_link"/>
-			<axis xyz="0 0 1"/>
-		</joint>
 		<!--***************************** back-left ****************************** -->
 		<xacro:if value="${enable_master}">

File: manipulator/AgileX/agilex_aloha_description/xacro/base/tracer.xacro (robot description, xacro)
@@ -2,4 +2,6 @@
 <robot name="tracer" xmlns:xacro="http://ros.org/wiki/xacro">
 	<link name="base_footprint"/>
+	<xacro:property name="PI" value="3.1415926535897931"/>
+	<xacro:property name="caster_height" value="0.0413"/>
 	<joint name="base_joint" type="fixed">
 		<origin xyz="0 0 0.143"/>
@@ -33,5 +35,4 @@
 	</link>
 	<joint name="inertial_joint" type="fixed">
-		<origin/>
 		<parent link="base_link"/>
 		<child link="inertial_link"/>
@@ -48,6 +49,7 @@
 		</visual>
 		<collision>
-			<geometry>
-				<mesh filename="file://$(find agilex_aloha_description)/meshes/tracer/tracer_wheel.obj"/>
+			<origin rpy="${PI/2} 0 0"/>
+			<geometry>
+				<cylinder radius="0.0607" length="0.0588"/>
 			</geometry>
 		</collision>
@@ -70,6 +72,7 @@
 		</visual>
 		<collision>
-			<geometry>
-				<mesh filename="file://$(find agilex_aloha_description)/meshes/tracer/tracer_wheel.obj"/>
+			<origin rpy="${PI/2} 0 0"/>
+			<geometry>
+				<cylinder radius="0.0607" length="0.0588"/>
 			</geometry>
 		</collision>
@@ -95,5 +98,5 @@
 		<parent link="base_link"/>
 		<child link="fl_castor_link"/>
-		<origin xyz="0.19 0.17 -0.038" rpy="-1.57 0 0"/>
+		<origin xyz="0.19 0.17 -${caster_height}" rpy="-${PI/2} 0 0"/>
 		<axis xyz="0 1 0"/>
 	</joint>
@@ -110,5 +113,5 @@
 	</link>
 	<joint name="fr_castor_wheel" type="continuous">
-		<origin xyz="0.18955 -0.17 -0.0380886" rpy="-1.57 0 0"/>
+		<origin xyz="0.18955 -0.17 -${caster_height}" rpy="-${PI/2} 0 0"/>
 		<parent link="base_link"/>
 		<child link="fr_castor_link"/>
@@ -127,5 +130,5 @@
 	</link>
 	<joint name="rr_castor_wheel" type="continuous">
-		<origin xyz="-0.18955 -0.17 -0.0380886" rpy="-1.57 0 0"/>
+		<origin xyz="-0.18955 -0.17 -${caster_height}" rpy="-${PI/2} 0 0"/>
 		<parent link="base_link"/>
 		<child link="rr_castor_link"/>
@@ -144,5 +147,5 @@
 	</link>
 	<joint name="rl_castor_wheel" type="continuous">
-		<origin xyz="-0.18955 0.17 -0.0380886" rpy="-1.57 0 0"/>
+		<origin xyz="-0.18955 0.17 -${caster_height}" rpy="-${PI/2} 0 0"/>
 		<parent link="base_link"/>
 		<child link="rl_castor_link"/>
@@ -160,6 +163,6 @@
 		</visual>
 		<collision>
-			<geometry>-->
-				<mesh filename="file://$(find agilex_aloha_description)/meshes/tracer/castor.obj"/>
+			<geometry>
+				<cylinder radius="0.0375" length="0.0534"/>
 			</geometry>
 		</collision>
@@ -183,6 +186,6 @@
 		</visual>
 		<collision>
-			<geometry>-->
-				<mesh filename="file://$(find agilex_aloha_description)/meshes/tracer/castor.obj"/>
+			<geometry>
+				<cylinder radius="0.0375" length="0.0534"/>
 			</geometry>
 		</collision>
@@ -207,5 +210,5 @@
 		<collision>
 			<geometry>
-				<mesh filename="file://$(find agilex_aloha_description)/meshes/tracer/castor.obj"/>
+				<cylinder radius="0.0375" length="0.0534"/>
 			</geometry>
 		</collision>
@@ -230,5 +233,5 @@
 		<collision>
 			<geometry>
-				<mesh filename="file://$(find agilex_aloha_description)/meshes/tracer/castor.obj"/>
+				<cylinder radius="0.0375" length="0.0534"/>
 			</geometry>
 		</collision>

File: manipulator/AgileX/agilex_aloha_description/xacro/base/tracer_v2.xacro (robot description, xacro)
@@ -113,5 +113,5 @@
 	</link>
 	<joint name="right_front_joint" type="fixed">
-		<origin xyz="0.23918 -0.1977 -0.058" rpy="3.1416 0 0"/>
+		<origin xyz="0.23918 -0.1977 -0.058"/>
 		<parent link="base_link"/>
 		<child link="right_front_link"/>
@@ -140,6 +140,6 @@
 		</collision>
 	</link>
-	<joint name="right_rea_joint" type="fixed">
-		<origin xyz="-0.27082 -0.183 -0.058" rpy="3.1416 0 0"/>
+	<joint name="right_rear_joint" type="fixed">
+		<origin xyz="-0.27082 -0.183 -0.058"/>
 		<parent link="base_link"/>
 		<child link="right_rear_link"/>

File: manipulator/AgileX/agilex_aloha_description/xacro/component.xacro (robot description, xacro)
@@ -4,5 +4,5 @@
 <!-- |    This file includes the base robot structure and both arms                    | -->
 <!-- =================================================================================== -->
-<robot name="LeftArm" xmlns:xacro="http://www.ros.org/wiki/xacro">
+<robot name="Agilex_Aloha_V1" xmlns:xacro="http://www.ros.org/wiki/xacro">
 	<xacro:arg name="type" default="ranger_mini"/>
 	<xacro:if value="${'$(arg type)' == 'ranger_mini'}">
@@ -15,3 +15,15 @@
 		<xacro:include filename="$(find agilex_aloha_description)/xacro/base/tracer_v2.xacro"/>
 	</xacro:if>
+	<xacro:if value="${'$(arg type)' == 'body_v1'}">
+		<link name="base_footprint"/>
+		<link name="left_base_link"/>
+		<link name="right_base_link"/>
+		<xacro:include filename="$(find agilex_aloha_description)/xacro/body/v1.xacro"/>
+	</xacro:if>
+	<xacro:if value="${'$(arg type)' == 'body_v2'}">
+		<link name="base_footprint"/>
+		<link name="left_base_link"/>
+		<link name="right_base_link"/>
+		<xacro:include filename="$(find agilex_aloha_description)/xacro/body/v2.xacro"/>
+	</xacro:if>
 </robot>
