Commit message: agilex split aloha  mesh clean up

File: humanoid/Galaxea/galaxea_r1_description/xacro/chassis.xacro (robot description, xacro)
@@ -60,6 +60,7 @@
       </visual>
       <collision>
+        <origin rpy="${PI/2} 0 0"/>
         <geometry>
-          <mesh filename="file://$(find galaxea_r1_description)/meshes/wheel_motor.obj"/>
+          <cylinder radius="0.07" length="0.048"/>
         </geometry>
       </collision>
@@ -113,6 +114,7 @@
       </visual>
       <collision>
+        <origin rpy="${PI/2} 0 0"/>
         <geometry>
-          <mesh filename="file://$(find galaxea_r1_description)/meshes/wheel_motor.obj"/>
+          <cylinder radius="0.07" length="0.048"/>
         </geometry>
       </collision>
@@ -164,6 +166,7 @@
       </visual>
       <collision>
+        <origin rpy="${PI/2} 0 0"/>
         <geometry>
-          <mesh filename="file://$(find galaxea_r1_description)/meshes/wheel_motor.obj"/>
+          <cylinder radius="0.07" length="0.048"/>
         </geometry>
       </collision>

File: manipulator/AgileX/agilex_aloha_description/xacro/aloha_split.xacro (robot description, xacro)
@@ -3,157 +3,6 @@
   <xacro:include filename="$(find agilex_aloha_description)/xacro/base/ranger_mini.xacro"/>
   <xacro:include filename="$(find piper_description)/xacro/Piper.xacro"/>
-  <link name="box_link">
-    <inertial>
-      <origin xyz="0.10921 -0.0087718 0.52779"/>
-      <mass value="27.261"/>
-      <inertia
-          ixx="1.8122"
-          ixy="4.558E-05"
-          ixz="0.014722"
-          iyy="1.7779"
-          iyz="-4.0693E-05"
-          izz="0.28053"/>
-    </inertial>
-    <visual>
-      <geometry>
-        <mesh filename="file://$(find agilex_aloha_description)/meshes/aloha_split/box_link.obj"/>
-      </geometry>
-    </visual>
-    <collision>
-      <geometry>
-        <mesh filename="file://$(find agilex_aloha_description)/meshes/aloha_split/box_link.obj"/>
-      </geometry>
-    </collision>
-  </link>
-  <joint name="box_joint" type="fixed">
-    <parent link="base"/>
-    <child link="box_link"/>
-  </joint>
-  <link name="front_camera_link">
-    <inertial>
-      <origin xyz="-0.011443 0.0003607 -0.0012124"/>
-      <mass value="0.020053"/>
-      <inertia
-          ixx="1.1182E-05"
-          ixy="2.589E-09"
-          ixz="5.6552E-08"
-          iyy="2.2729E-06"
-          iyz="-6.7447E-07"
-          izz="1.0081E-05"/>
-    </inertial>
-    <visual>
-      <geometry>
-        <mesh filename="file://$(find sensor_models)/meshes/dabai/dabai.obj"/>
-      </geometry>
-    </visual>
-  </link>
-  <joint name="front_camera_joint" type="fixed">
-    <origin xyz="0.35679 0 0.15819" rpy="0 0.6606 -0.0051043"/>
-    <parent link="box_link"/>
-    <child link="front_camera_link"/>
-  </joint>
-  <link name="lidar_link">
-    <inertial>
-      <origin xyz="-0.0022133 -0.00090659 0.025996"/>
-      <mass value="0.048617"/>
-      <inertia
-          ixx="1.0358E-05"
-          ixy="9.2377E-09"
-          ixz="-2.6386E-07"
-          iyy="1.0387E-05"
-          iyz="-2.6377E-07"
-          izz="1.7919E-05"/>
-    </inertial>
-    <visual>
-      <geometry>
-        <mesh filename="file://$(find sensor_models)/meshes/mid360/mid360.obj"/>
-      </geometry>
-    </visual>
-  </link>
-  <joint name="lidar_joint" type="fixed">
-    <origin xyz="0.31755 0 0.036188"/>
-    <parent link="box_link"/>
-    <child link="lidar_link"/>
-  </joint>
-  <link name="lifting_link">
-    <inertial>
-      <origin xyz="0.071327 0.00032985 0.10599"/>
-      <mass value="0.47066"/>
-      <inertia
-          ixx="0.010952"
-          ixy="-5.2124E-06"
-          ixz="-0.00046317"
-          iyy="0.0018329"
-          iyz="-4.6428E-06"
-          izz="0.010201"/>
-    </inertial>
-    <visual>
-      <geometry>
-        <mesh filename="file://$(find agilex_aloha_description)/meshes/aloha_split/lift_link.obj"/>
-      </geometry>
-    </visual>
-    <collision>
-      <geometry>
-        <mesh filename="file://$(find agilex_aloha_description)/meshes/aloha_split/lift_link.obj"/>
-      </geometry>
-    </collision>
-  </link>
-  <joint name="lifting_joint" type="prismatic">
-    <origin xyz="0.22448 0 1.1147"/>
-    <parent link="box_link"/>
-    <child link="lifting_link"/>
-    <axis xyz="0 0 1"/>
-    <limit lower="-0.6" upper="0.0" effort="1000" velocity="10.0"/>
-  </joint>
-  <link name="top_camera_link">
-    <inertial>
-      <origin xyz="-0.011443 2.4833E-05 -0.0012615"/>
-      <mass value="0.020053"/>
-      <inertia
-          ixx="1.1181E-05"
-          ixy="1.204E-07"
-          ixz="4.9068E-08"
-          iyy="2.2587E-06"
-          iyz="5.7637E-07"
-          izz="1.0097E-05"/>
-    </inertial>
-    <visual>
-      <geometry>
-        <mesh filename="file://$(find sensor_models)/meshes/dabai/dabai.obj"/>
-      </geometry>
-    </visual>
-  </link>
-  <joint name="top_camera_joint" type="fixed">
-    <origin xyz="0.16194 0 0.29838" rpy="0 0.00080758 -0.01623"/>
-    <parent link="lifting_link"/>
-    <child link="top_camera_link"/>
-  </joint>
-  <link name="top_camera_support">
-    <visual>
-      <geometry>
-        <mesh filename="file://$(find agilex_aloha_description)/meshes/aloha_split/camera_support.obj"/>
-      </geometry>
-    </visual>
-  </link>
-  <joint name="top_camera_support_joint" type="fixed">
-    <origin xyz="0.16194 0 0.29838" rpy="0 0.00080758 -0.01623"/>
-    <parent link="lifting_link"/>
-    <child link="top_camera_support"/>
-  </joint>
+  <xacro:include filename="$(find agilex_aloha_description)/xacro/body/split.xacro"/>
   <xacro:Piper name="left"/>
-  <joint name="arm_and_lifting_left" type="fixed">
-    <origin xyz="0.144 0.306 0.138"/>
-    <parent link="lifting_link"/>
-    <child link="left_base_link"/>
-    <axis xyz="0.0 0.0 0.0"/>
-    <limit lower="0.0" upper="0.0" effort="0.0" velocity="0.0"/>
-  </joint>
   <xacro:Piper name="right"/>
-  <joint name="arm_and_lifting_right" type="fixed">
-    <origin xyz="0.144 -0.306 0.138"/>
-    <parent link="lifting_link"/>
-    <child link="right_base_link"/>
-    <axis xyz="0.0 0.0 0.0"/>
-    <limit lower="0.0" upper="0.0" effort="0.0" velocity="0.0"/>
-  </joint>
 </robot>

File: manipulator/AgileX/agilex_aloha_description/xacro/base/tracer_v2.xacro (robot description, xacro)
@@ -1,5 +1,6 @@
 <?xml version="1.0" encoding="utf-8"?>
-<robot name="tracer2">
+<robot name="tracer2" xmlns:xacro="http://ros.org/wiki/xacro">
 	<link name="base_footprint"/>
+	<xacro:property name="PI" value="3.1415926535897931"/>
 	<joint name="base_joint" type="fixed">
 		<origin xyz="0 0 0.15"/>
@@ -49,6 +50,7 @@
 		</visual>
 		<collision>
-			<geometry>
-				<mesh filename="file://$(find agilex_aloha_description)/meshes/tracer_v2/drive_wheel.obj"/>
+			<origin xyz="0 0 -0.0048"/>
+			<geometry>
+				<cylinder radius="0.0628" length="0.04"/>
 			</geometry>
 		</collision>
@@ -78,6 +80,7 @@
 		</visual>
 		<collision>
-			<geometry>
-				<mesh filename="file://$(find agilex_aloha_description)/meshes/tracer_v2/drive_wheel.obj"/>
+			<origin xyz="0 0 -0.0048" />
+			<geometry>
+				<cylinder radius="0.0628" length="0.04"/>
 			</geometry>
 		</collision>
@@ -87,5 +90,5 @@
 		<parent link="base_link"/>
 		<child link="left_Link"/>
-		<axis xyz="0 0 1"/>
+		<axis xyz="0 0 -1"/>
 	</joint>
 	<link name="right_front_link">
@@ -106,14 +109,23 @@
 			</geometry>
 		</visual>
-		<collision>
-			<geometry>
-				<mesh filename="file://$(find agilex_aloha_description)/meshes/tracer_v2/support_wheel.obj"/>
-			</geometry>
-		</collision>
-	</link>
-	<joint name="right_front_joint" type="fixed">
+	</link>
+	<joint name="right_front_joint" type="continuous">
 		<origin xyz="0.23918 -0.1977 -0.058"/>
 		<parent link="base_link"/>
 		<child link="right_front_link"/>
+		<axis xyz="0 0 1"/>
+	</joint>
+	<link name="right_front_wheel">
+		<collision>
+			<geometry>
+				<cylinder radius="0.0375" length="0.048"/>
+			</geometry>
+		</collision>
+	</link>
+	<joint name="right_front_wheel_joint" type="continuous">
+		<origin xyz="-0.02 0 -0.0575" rpy="${PI/2} 0 0"/>
+		<parent link="right_front_link"/>
+		<child link="right_front_wheel"/>
+		<axis xyz="0 0 1"/>
 	</joint>
 	<link name="right_rear_link">
@@ -134,14 +146,23 @@
 			</geometry>
 		</visual>
-		<collision>
-			<geometry>
-				<mesh filename="file://$(find agilex_aloha_description)/meshes/tracer_v2/support_wheel.obj"/>
-			</geometry>
-		</collision>
-	</link>
-	<joint name="right_rear_joint" type="fixed">
+	</link>
+	<joint name="right_rear_joint" type="continuous">
 		<origin xyz="-0.27082 -0.183 -0.058"/>
 		<parent link="base_link"/>
 		<child link="right_rear_link"/>
+		<axis xyz="0 0 1"/>
+	</joint>
+	<link name="right_rear_wheel">
+		<collision>
+			<geometry>
+				<cylinder radius="0.0375" length="0.048"/>
+			</geometry>
+		</collision>
+	</link>
+	<joint name="right_rear_wheel_joint" type="continuous">
+		<origin xyz="-0.02 0 -0.0575" rpy="${PI/2} 0 0"/>
+		<parent link="right_rear_link"/>
+		<child link="right_rear_wheel"/>
+		<axis xyz="0 0 1"/>
 	</joint>
 	<link name="left_front_link">
@@ -162,14 +183,23 @@
 			</geometry>
 		</visual>
-		<collision>
-			<geometry>
-				<mesh filename="file://$(find agilex_aloha_description)/meshes/tracer_v2/support_wheel.obj"/>
-			</geometry>
-		</collision>
-	</link>
-	<joint name="left_front_joint" type="fixed">
+	</link>
+	<joint name="left_front_joint" type="continuous">
 		<origin xyz="0.23918 0.1977 -0.058"/>
 		<parent link="base_link"/>
 		<child link="left_front_link"/>
+		<axis xyz="0 0 1"/>
+	</joint>
+	<link name="left_front_wheel">
+		<collision>
+			<geometry>
+				<cylinder radius="0.0375" length="0.048"/>
+			</geometry>
+		</collision>
+	</link>
+	<joint name="left_front_wheel_joint" type="continuous">
+		<origin xyz="-0.02 0 -0.0575" rpy="${PI/2} 0 0"/>
+		<parent link="left_front_link"/>
+		<child link="left_front_wheel"/>
+		<axis xyz="0 0 1"/>
 	</joint>
 	<link name="left_rear_link">
@@ -189,14 +219,23 @@
 			</geometry>
 		</visual>
-		<collision>
-			<geometry>
-				<mesh filename="file://$(find agilex_aloha_description)/meshes/tracer_v2/support_wheel.obj"/>
-			</geometry>
-		</collision>
-	</link>
-	<joint name="left_rear_joint" type="fixed">
+	</link>
+	<joint name="left_rear_joint" type="continuous">
 		<origin xyz="-0.27077 0.18305 -0.058"/>
 		<parent link="base_link"/>
 		<child link="left_rear_link"/>
+		<axis xyz="0 0 1"/>
+	</joint>
+	<link name="left_rear_wheel">
+		<collision>
+			<geometry>
+				<cylinder radius="0.0375" length="0.048"/>
+			</geometry>
+		</collision>
+	</link>
+	<joint name="left_rear_wheel_joint" type="continuous">
+		<origin xyz="-0.02 0 -0.0575" rpy="${PI/2} 0 0"/>
+		<parent link="left_rear_link"/>
+		<child link="left_rear_wheel"/>
+		<axis xyz="0 0 1"/>
 	</joint>
 </robot>

File: manipulator/AgileX/agilex_aloha_description/xacro/component.xacro (robot description, xacro)
@@ -4,5 +4,5 @@
 <!-- |    This file includes the base robot structure and both arms                    | -->
 <!-- =================================================================================== -->
-<robot name="Agilex_Aloha_V1" xmlns:xacro="http://www.ros.org/wiki/xacro">
+<robot name="Agilex_Aloha_Spilt" xmlns:xacro="http://www.ros.org/wiki/xacro">
 	<xacro:arg name="type" default="ranger_mini"/>
 	<xacro:if value="${'$(arg type)' == 'ranger_mini'}">
@@ -27,3 +27,9 @@
 		<xacro:include filename="$(find agilex_aloha_description)/xacro/body/v2.xacro"/>
 	</xacro:if>
+	<xacro:if value="${'$(arg type)' == 'body_split'}">
+		<link name="base"/>
+		<link name="left_base_link"/>
+		<link name="right_base_link"/>
+		<xacro:include filename="$(find agilex_aloha_description)/xacro/body/split.xacro"/>
+	</xacro:if>
 </robot>
