Commit message: add arx wheel

File: humanoid/ARX/arx_lift_description/xacro/mobile_base.xacro (robot description, xacro)
@@ -1,4 +1,5 @@
 <?xml version="1.0" encoding="utf-8"?>
 <robot xmlns:xacro="http://www.ros.org/wiki/xacro">
+  <xacro:property name="PI" value="3.1415926535897931"/>
   <xacro:macro name="MobileBase">
     <link name="base_link"/>
@@ -31,4 +32,9 @@
         <inertia ixx="0.008031" ixy="-0.002428" ixz="0.0" iyy="0.010834" iyz="0.0" izz="0.006629"/>
       </inertial>
+      <visual>
+        <geometry>
+          <mesh filename="file://$(find arx_lift_description)/meshes/wheel.obj"/>
+        </geometry>
+      </visual>
     </link>
     <link name="wheel_2">
@@ -38,4 +44,9 @@
         <inertia ixx="0.008031" ixy="0.002428" ixz="-0.0" iyy="0.010834" iyz="0.0" izz="0.006629"/>
       </inertial>
+      <visual>
+        <geometry>
+          <mesh filename="file://$(find arx_lift_description)/meshes/wheel.obj"/>
+        </geometry>
+      </visual>
     </link>
     <link name="wheel_3">
@@ -45,21 +56,27 @@
         <inertia ixx="0.012235" ixy="-0.0" ixz="0.0" iyy="0.006629" iyz="0.0" izz="0.006629"/>
       </inertial>
+      <visual>
+        <geometry>
+          <mesh filename="file://$(find arx_lift_description)/meshes/wheel.obj"/>
+        </geometry>
+      </visual>
     </link>
-    <joint name="joint_wheel1" type="fixed">
-      <origin xyz="-0.182349 0.315838 0.03"/>
+    <joint name="joint_wheel1" type="continuous">
+      <origin xyz="-0.182349 0.315838 0.03" rpy="0.0 0.0 ${-PI/3}"/>
       <parent link="base"/>
       <child link="wheel_1"/>
+      <axis xyz="1 0 0"/>
     </joint>
-    <joint name="joint_wheel2" type="fixed">
-      <origin xyz="-0.182349 -0.315838 0.03"/>
+    <joint name="joint_wheel2" type="continuous">
+      <origin xyz="-0.182349 -0.315838 0.03" rpy="0.0 0.0 ${PI/3}"/>
       <parent link="base"/>
       <child link="wheel_2"/>
-      <axis xyz="-0.5 -0.866025 0.0"/>
+      <axis xyz="1 0 0"/>
     </joint>
-    <joint name="joint_wheel3" type="fixed">
-      <origin xyz="0.364699 0.0 0.03"/>
+    <joint name="joint_wheel3" type="continuous" >
+      <origin xyz="0.364699 0.0 0.03" rpy="0.0 0.0 ${PI}"/>
       <parent link="base"/>
       <child link="wheel_3"/>
-      <axis xyz="1.0 0.0 -0.0"/>
+      <axis xyz="1 0 0"/>
     </joint>
   </xacro:macro>
