Commit message: Dexfoce w1 (#15)
* add dexforce w1 ros2 control

* add brainco revo2 config

* update mesh to glb for astribot s1

* agibot g1 update mesh to glb

* add zerith h1

* zerith h1 mesh cleaned

* add angellun omniwheel

* using angellun omniwheel

* remove arx and using submodules

* remove arx and using submodules

* remove Ubtech and add as submodule from robot-descriptions-ubtech

* update readme

* update readme

File: humanoid/Agibot/agibot_g1_description/urdf/agibot_g1.urdf (robot description, URDF)
Before this commit: robot Agibot G1, 30 links, 29 joints
Links:
- link base_link: geometry collision box size=0.29833984 0.3376392 1.0; collision box size=0.5796094 0.449 0.27073438
- link body_link1: geometry collision box size=0.16064453 0.05555534399999999 0.1328125; collision box size=0.16259765999999998 0.04375648500000001 0.16015625
- link body_link2: geometry collision box size=0.34570312 0.18107724 0.3125; collision cylinder length=0.08697056999999997 radius=0.09662318
- link head_link1: geometry visual mesh filename=package://agibot_g1_description/meshes/base/head_link1.glb
- link head_link2: geometry collision sphere radius=0.11257068650657154; visual mesh filename=package://agibot_g1_description/meshes/base/head_link2.glb
- link left_base_link: geometry visual mesh filename=package://agibot_g1_description/meshes/arm/base_link.glb
- link left_end_link: geometry collision cylinder length=0.045999998692423105 radius=0.030799950382754494; visual mesh filename=package://agibot_g1_description/meshes/arm/link7.glb
- link left_link1: geometry collision cylinder length=0.16642063483595848 radius=0.05579268228774888; visual mesh filename=package://agibot_g1_description/meshes/arm/link1.glb
- link left_link2: geometry collision cylinder length=0.18085919 radius=0.06302423; visual mesh filename=package://agibot_g1_description/meshes/arm/link2.glb
- link left_link3: geometry collision cylinder length=0.22061403840780258 radius=0.05216156143823925; visual mesh filename=package://agibot_g1_description/meshes/arm/link3.glb
- link left_link4: geometry collision cylinder length=0.154955404 radius=0.057891708; visual mesh filename=package://agibot_g1_description/meshes/arm/link4.glb
- link left_link5: geometry collision cylinder length=0.13423806056380272 radius=0.04562028545392604; visual mesh filename=package://agibot_g1_description/meshes/arm/link5.glb
- link left_link6: geometry collision cylinder length=0.18272488500982115 radius=0.04857149291994264; visual mesh filename=package://agibot_g1_description/meshes/arm/link6.glb
- link right_base_link: geometry visual mesh filename=package://agibot_g1_description/meshes/arm/base_link.glb
- link right_end_link: geometry collision cylinder length=0.045999998692423105 radius=0.030799950382754494; visual mesh filename=package://agibot_g1_description/meshes/arm/link7.glb
- link right_link1: geometry collision cylinder length=0.16642063483595848 radius=0.05579268228774888; visual mesh filename=package://agibot_g1_description/meshes/arm/link1.glb
- link right_link2: geometry collision cylinder length=0.18085919 radius=0.06302423; visual mesh filename=package://agibot_g1_description/meshes/arm/link2.glb
- link right_link3: geometry collision cylinder length=0.22061403840780258 radius=0.05216156143823925; visual mesh filename=package://agibot_g1_description/meshes/arm/link3.glb
- link right_link4: geometry collision cylinder length=0.154955404 radius=0.057891708; visual mesh filename=package://agibot_g1_description/meshes/arm/link4.glb
- link right_link5: geometry collision cylinder length=0.13423806056380272 radius=0.04562028545392604; visual mesh filename=package://agibot_g1_description/meshes/arm/link5.glb
- link right_link6: geometry collision cylinder length=0.18272488500982115 radius=0.04857149291994264; visual mesh filename=package://agibot_g1_description/meshes/arm/link6.glb

File: humanoid/Agibot/agibot_g1_description/urdf/agibot_g1_omni-picker.urdf (robot description, URDF)
Before this commit: robot Agibot G1, 30 links, 29 joints
Links:
- link base_link: geometry collision box size=0.29833984 0.3376392 1.0; collision box size=0.5796094 0.449 0.27073438
- link body_link1: geometry collision box size=0.16064453 0.05555534399999999 0.1328125; collision box size=0.16259765999999998 0.04375648500000001 0.16015625
- link body_link2: geometry collision box size=0.34570312 0.18107724 0.3125; collision cylinder length=0.08697056999999997 radius=0.09662318
- link head_link1: geometry visual mesh filename=package://agibot_g1_description/meshes/base/head_link1.glb
- link head_link2: geometry collision sphere radius=0.11257068650657154; visual mesh filename=package://agibot_g1_description/meshes/base/head_link2.glb
- link left_base_link: geometry visual mesh filename=package://agibot_g1_description/meshes/arm/base_link.glb
- link left_end_link: geometry collision cylinder length=0.045999998692423105 radius=0.030799950382754494; visual mesh filename=package://agibot_g1_description/meshes/arm/link7.glb
- link left_link1: geometry collision cylinder length=0.16642063483595848 radius=0.05579268228774888; visual mesh filename=package://agibot_g1_description/meshes/arm/link1.glb
- link left_link2: geometry collision cylinder length=0.18085919 radius=0.06302423; visual mesh filename=package://agibot_g1_description/meshes/arm/link2.glb
- link left_link3: geometry collision cylinder length=0.22061403840780258 radius=0.05216156143823925; visual mesh filename=package://agibot_g1_description/meshes/arm/link3.glb
- link left_link4: geometry collision cylinder length=0.154955404 radius=0.057891708; visual mesh filename=package://agibot_g1_description/meshes/arm/link4.glb
- link left_link5: geometry collision cylinder length=0.13423806056380272 radius=0.04562028545392604; visual mesh filename=package://agibot_g1_description/meshes/arm/link5.glb
- link left_link6: geometry collision cylinder length=0.18272488500982115 radius=0.04857149291994264; visual mesh filename=package://agibot_g1_description/meshes/arm/link6.glb
- link right_base_link: geometry visual mesh filename=package://agibot_g1_description/meshes/arm/base_link.glb
- link right_end_link: geometry collision cylinder length=0.045999998692423105 radius=0.030799950382754494; visual mesh filename=package://agibot_g1_description/meshes/arm/link7.glb
- link right_link1: geometry collision cylinder length=0.16642063483595848 radius=0.05579268228774888; visual mesh filename=package://agibot_g1_description/meshes/arm/link1.glb
- link right_link2: geometry collision cylinder length=0.18085919 radius=0.06302423; visual mesh filename=package://agibot_g1_description/meshes/arm/link2.glb
- link right_link3: geometry collision cylinder length=0.22061403840780258 radius=0.05216156143823925; visual mesh filename=package://agibot_g1_description/meshes/arm/link3.glb
- link right_link4: geometry collision cylinder length=0.154955404 radius=0.057891708; visual mesh filename=package://agibot_g1_description/meshes/arm/link4.glb
- link right_link5: geometry collision cylinder length=0.13423806056380272 radius=0.04562028545392604; visual mesh filename=package://agibot_g1_description/meshes/arm/link5.glb
- link right_link6: geometry collision cylinder length=0.18272488500982115 radius=0.04857149291994264; visual mesh filename=package://agibot_g1_description/meshes/arm/link6.glb

File: humanoid/Agibot/agibot_g1_description/xacro/120s_camera_stand.xacro (robot description, xacro)
@@ -10,5 +10,5 @@
 			<visual>
 				<geometry>
-					<mesh filename="file://$(find agibot_g1_description)/meshes/camera/120s_camera_stand.obj"/>
+					<mesh filename="file://$(find agibot_g1_description)/meshes/camera/120s_camera_stand.glb"/>
 				</geometry>
 			</visual>

File: humanoid/Agibot/agibot_g1_description/xacro/g1_arm.xacro (robot description, xacro)
@@ -13,5 +13,5 @@
 			<visual>
 				<geometry>
-					<mesh filename="file://$(find agibot_g1_description)/meshes/arm/base_link.obj"/>
+					<mesh filename="file://$(find agibot_g1_description)/meshes/arm/base_link.glb"/>
 				</geometry>
 			</visual>
@@ -27,5 +27,5 @@
 			<visual>
 				<geometry>
-					<mesh filename="file://$(find agibot_g1_description)/meshes/arm/link1.obj"/>
+					<mesh filename="file://$(find agibot_g1_description)/meshes/arm/link1.glb"/>
 				</geometry>
 			</visual>
@@ -47,5 +47,5 @@
 			<visual>
 				<geometry>
-					<mesh filename="file://$(find agibot_g1_description)/meshes/arm/link2.obj"/>
+					<mesh filename="file://$(find agibot_g1_description)/meshes/arm/link2.glb"/>
 				</geometry>
 			</visual>
@@ -65,5 +65,5 @@
 			<visual>
 				<geometry>
-					<mesh filename="file://$(find agibot_g1_description)/meshes/arm/link3.obj"/>
+					<mesh filename="file://$(find agibot_g1_description)/meshes/arm/link3.glb"/>
 				</geometry>
 			</visual>
@@ -83,5 +83,5 @@
 			<visual>
 				<geometry>
-					<mesh filename="file://$(find agibot_g1_description)/meshes/arm/link4.obj"/>
+					<mesh filename="file://$(find agibot_g1_description)/meshes/arm/link4.glb"/>
 				</geometry>
 			</visual>
@@ -102,5 +102,5 @@
 			<visual>
 				<geometry>
-					<mesh filename="file://$(find agibot_g1_description)/meshes/arm/link5.obj"/>
+					<mesh filename="file://$(find agibot_g1_description)/meshes/arm/link5.glb"/>
 				</geometry>
 			</visual>
@@ -121,5 +121,5 @@
 			<visual>
 				<geometry>
-					<mesh filename="file://$(find agibot_g1_description)/meshes/arm/link6.obj"/>
+					<mesh filename="file://$(find agibot_g1_description)/meshes/arm/link6.glb"/>
 				</geometry>
 			</visual>
@@ -140,5 +140,5 @@
 			<visual>
 				<geometry>
-					<mesh filename="file://$(find agibot_g1_description)/meshes/arm/link7.obj"/>
+					<mesh filename="file://$(find agibot_g1_description)/meshes/arm/link7.glb"/>
 				</geometry>
 			</visual>

File: humanoid/Agibot/agibot_g1_description/xacro/g1_base.xacro (robot description, xacro)
@@ -21,5 +21,5 @@
 		<visual>
 			<geometry>
-				<mesh filename="file://$(find agibot_g1_description)/meshes/base/base.obj"/>
+				<mesh filename="file://$(find agibot_g1_description)/meshes/base/base.glb"/>
 			</geometry>
 		</visual>
@@ -75,5 +75,5 @@
 		<visual>
 			<geometry>
-				<mesh filename="file://$(find agibot_g1_description)/meshes/base/wheel.obj" scale="1 1 1"/>
+				<mesh filename="file://$(find agibot_g1_description)/meshes/base/wheel.glb" scale="1 1 1"/>
 			</geometry>
 		</visual>
@@ -117,5 +117,5 @@
 		<visual>
 			<geometry>
-				<mesh filename="file://$(find agibot_g1_description)/meshes/base/wheel.obj" scale="1 -1 1"/>
+				<mesh filename="file://$(find agibot_g1_description)/meshes/base/wheel.glb" scale="1 -1 1"/>
 			</geometry>
 		</visual>
@@ -142,5 +142,5 @@
 		<visual>
 			<geometry>
-				<mesh filename="file://$(find agibot_g1_description)/meshes/base/body_link1.obj"/>
+				<mesh filename="file://$(find agibot_g1_description)/meshes/base/body_link1.glb"/>
 			</geometry>
 		</visual>
@@ -172,5 +172,5 @@
 		<visual>
 			<geometry>
-				<mesh filename="file://$(find agibot_g1_description)/meshes/base/body_link2.obj"/>
+				<mesh filename="file://$(find agibot_g1_description)/meshes/base/body_link2.glb"/>
 			</geometry>
 			<origin rpy="0.0 0.0 -1.5707963267948966"/>
@@ -213,5 +213,5 @@
 		<visual>
 			<geometry>
-				<mesh filename="file://$(find agibot_g1_description)/meshes/base/head_link1.obj"/>
+				<mesh filename="file://$(find agibot_g1_description)/meshes/base/head_link1.glb"/>
 			</geometry>
 		</visual>
@@ -226,5 +226,5 @@
 		<visual>
 			<geometry>
-				<mesh filename="file://$(find agibot_g1_description)/meshes/base/head_link2.obj"/>
+				<mesh filename="file://$(find agibot_g1_description)/meshes/base/head_link2.glb"/>
 			</geometry>
 			<origin rpy="-3.141592653589793 0.0 0.0"/>

File: humanoid/Agibot/agibot_g1_description/xacro/omnipicker_camera_stand.xacro (robot description, xacro)
@@ -11,5 +11,5 @@
 			<visual>
 				<geometry>
-					<mesh filename="file://$(find agibot_g1_description)/meshes/camera/omni_picker_camera_stand.obj"/>
+					<mesh filename="file://$(find agibot_g1_description)/meshes/camera/omnipicker_camera_stand.glb"/>
 				</geometry>
 			</visual>

File: humanoid/Agibot/agibot_omni_description/xacro/omni_picker.xacro (robot description, xacro)
@@ -13,5 +13,5 @@
 			<visual>
 				<geometry>
-					<mesh filename="${mesh_path}/gripper_base.obj"/>
+					<mesh filename="${mesh_path}/gripper_base.glb"/>
 				</geometry>
 			</visual>
@@ -31,10 +31,10 @@
 			<visual>
 				<geometry>
-					<mesh filename="${mesh_path}/narrow_1.obj"/>
-				</geometry>
-			</visual>
-			<collision>
-				<geometry>
-					<mesh filename="${mesh_path}/narrow_1.obj"/>
+					<mesh filename="${mesh_path}/narrow_1.glb"/>
+				</geometry>
+			</visual>
+			<collision>
+				<geometry>
+					<mesh filename="${mesh_path}/narrow_1.glb"/>
 				</geometry>
 			</collision>
@@ -61,10 +61,10 @@
 			<visual>
 				<geometry>
-					<mesh filename="${mesh_path}/narrow_2.obj"/>
-				</geometry>
-			</visual>
-			<collision>
-				<geometry>
-					<mesh filename="${mesh_path}/narrow_2.obj"/>
+					<mesh filename="${mesh_path}/narrow_2.glb"/>
+				</geometry>
+			</visual>
+			<collision>
+				<geometry>
+					<mesh filename="${mesh_path}/narrow_2.glb"/>
 				</geometry>
 			</collision>
@@ -92,10 +92,10 @@
 			<visual>
 				<geometry>
-					<mesh filename="${mesh_path}/narrow_3.obj"/>
-				</geometry>
-			</visual>
-			<collision>
-				<geometry>
-					<mesh filename="${mesh_path}/narrow_3.obj"/>
+					<mesh filename="${mesh_path}/narrow_3.glb"/>
+				</geometry>
+			</visual>
+			<collision>
+				<geometry>
+					<mesh filename="${mesh_path}/narrow_3.glb"/>
 				</geometry>
 			</collision>
@@ -131,10 +131,10 @@
 			<visual>
 				<geometry>
-					<mesh filename="${mesh_path}/narrow_loop.obj"/>
-				</geometry>
-			</visual>
-			<collision>
-				<geometry>
-					<mesh filename="${mesh_path}/narrow_loop.obj"/>
+					<mesh filename="${mesh_path}/narrow_loop.glb"/>
+				</geometry>
+			</visual>
+			<collision>
+				<geometry>
+					<mesh filename="${mesh_path}/narrow_loop.glb"/>
 				</geometry>
 			</collision>
@@ -162,10 +162,10 @@
 			<visual>
 				<geometry>
-					<mesh filename="${mesh_path}/wide_1.obj"/>
-				</geometry>
-			</visual>
-			<collision>
-				<geometry>
-					<mesh filename="${mesh_path}/wide_1.obj"/>
+					<mesh filename="${mesh_path}/wide_1.glb"/>
+				</geometry>
+			</visual>
+			<collision>
+				<geometry>
+					<mesh filename="${mesh_path}/wide_1.glb"/>
 				</geometry>
 			</collision>
@@ -193,10 +193,10 @@
 			<visual>
 				<geometry>
-					<mesh filename="${mesh_path}/wide_2.obj"/>
-				</geometry>
-			</visual>
-			<collision>
-				<geometry>
-					<mesh filename="${mesh_path}/wide_2.obj"/>
+					<mesh filename="${mesh_path}/wide_2.glb"/>
+				</geometry>
+			</visual>
+			<collision>
+				<geometry>
+					<mesh filename="${mesh_path}/wide_2.glb"/>
 				</geometry>
 			</collision>
@@ -224,10 +224,10 @@
 			<visual>
 				<geometry>
-					<mesh filename="${mesh_path}/wide_3.obj"/>
-				</geometry>
-			</visual>
-			<collision>
-				<geometry>
-					<mesh filename="${mesh_path}/wide_3.obj"/>
+					<mesh filename="${mesh_path}/wide_3.glb"/>
+				</geometry>
+			</visual>
+			<collision>
+				<geometry>
+					<mesh filename="${mesh_path}/wide_3.glb"/>
 				</geometry>
 			</collision>
@@ -261,10 +261,10 @@
 			<visual>
 				<geometry>
-					<mesh filename="${mesh_path}/wide_loop.obj"/>
-				</geometry>
-			</visual>
-			<collision>
-				<geometry>
-					<mesh filename="${mesh_path}/wide_loop.obj"/>
+					<mesh filename="${mesh_path}/wide_loop.glb"/>
+				</geometry>
+			</visual>
+			<collision>
+				<geometry>
+					<mesh filename="${mesh_path}/wide_loop.glb"/>
 				</geometry>
 			</collision>

File: humanoid/Astribot/astribot_s1_description/urdf/astribot_s1.urdf (robot description, URDF)
Before this commit: robot astribot_s1, 21 links, 20 joints
Links:
- link head_link_1: geometry visual mesh filename=package://astribot_s1_description/meshes/s1_head/link1.glb
- link head_link_2: geometry collision sphere radius=0.11; visual mesh filename=package://astribot_s1_description/meshes/s1_head/link2.glb
- link left_link_1: geometry visual mesh filename=package://astribot_s1_description/meshes/s1_arm/link1.glb
- link left_link_2: geometry visual mesh filename=package://astribot_s1_description/meshes/s1_arm/link2.glb
- link left_link_3: geometry collision cylinder length=0.18 radius=0.05; visual mesh filename=package://astribot_s1_description/meshes/s1_arm/link3.glb
- link left_link_4: geometry collision sphere radius=0.06; visual mesh filename=package://astribot_s1_description/meshes/s1_arm/link4.glb
- link left_link_5: geometry collision cylinder length=0.14 radius=0.05; visual mesh filename=package://astribot_s1_description/meshes/s1_arm/link5.glb
- link left_link_6: geometry visual mesh filename=package://astribot_s1_description/meshes/s1_arm/link6.glb
- link left_link_7: geometry collision sphere radius=0.05; visual mesh filename=package://astribot_s1_description/meshes/s1_arm/link7.glb
- link right_link_1: geometry visual mesh filename=package://astribot_s1_description/meshes/s1_arm/link1.glb scale=1 -1 1
- link right_link_2: geometry visual mesh filename=package://astribot_s1_description/meshes/s1_arm/link2.glb scale=1 1 -1
- link right_link_3: geometry collision cylinder length=0.18 radius=0.05; visual mesh filename=package://astribot_s1_description/meshes/s1_arm/link3.glb
- link right_link_4: geometry collision sphere radius=0.06; visual mesh filename=package://astribot_s1_description/meshes/s1_arm/link4.glb
- link right_link_5: geometry collision cylinder length=0.14 radius=0.05; visual mesh filename=package://astribot_s1_description/meshes/s1_arm/link5.glb
- link right_link_6: geometry visual mesh filename=package://astribot_s1_description/meshes/s1_arm/link6.glb
- link right_link_7: geometry collision sphere radius=0.05; visual mesh filename=package://astribot_s1_description/meshes/s1_arm/link7.glb
- link torso_link_1: geometry collision cylinder length=0.3 radius=0.1; visual mesh filename=package://astribot_s1_description/meshes/s1_torso/link1.glb
- link torso_link_2: geometry collision cylinder length=0.3 radius=0.1; visual mesh filename=package://astribot_s1_description/meshes/s1_torso/link2.glb
- link torso_link_3: geometry collision cylinder length=0.35 radius=0.09; visual mesh filename=package://astribot_s1_description/meshes/s1_torso/link3.glb
- link torso_link_4: geometry visual mesh filename=package://astribot_s1_description/meshes/s1_torso/link4.glb

File: humanoid/Astribot/astribot_s1_description/xacro/components/base.xacro (robot description, xacro)
@@ -15,5 +15,5 @@
 			<visual>
 				<geometry>
-					<mesh filename="file://$(find astribot_s1_description)/meshes/s1_torso/base.obj"/>
+					<mesh filename="file://$(find astribot_s1_description)/meshes/s1_torso/base.glb"/>
 				</geometry>
 			</visual>
@@ -24,5 +24,5 @@
 			</collision>
 		</link>
-		<xacro:include filename="$(find arx_lift_description)/xacro/components/wheel.xacro"/>
+		<xacro:include filename="$(find component_models)/xacro/angellun_omniwheel.xacro"/>
 		<!-- 根据enable_wheel_joints参数决定使用轮子宏还是空link -->
 		<xacro:if value="${enable_wheel_joints}">
@@ -90,5 +90,5 @@
 			<visual>
 				<geometry>
-					<mesh filename="file://$(find astribot_s1_description)/meshes/s1_torso/link1.obj"/>
+					<mesh filename="file://$(find astribot_s1_description)/meshes/s1_torso/link1.glb"/>
 				</geometry>
 				<material name="">
@@ -119,5 +119,5 @@
 			<visual>
 				<geometry>
-					<mesh filename="file://$(find astribot_s1_description)/meshes/s1_torso/link2.obj"/>
+					<mesh filename="file://$(find astribot_s1_description)/meshes/s1_torso/link2.glb"/>
 				</geometry>
 				<material name="">
@@ -149,5 +149,5 @@
 			<visual>
 				<geometry>
-					<mesh filename="file://$(find astribot_s1_description)/meshes/s1_torso/link3.obj"/>
+					<mesh filename="file://$(find astribot_s1_description)/meshes/s1_torso/link3.glb"/>
 				</geometry>
 			</visual>
@@ -177,5 +177,5 @@
 			<visual>
 				<geometry>
-					<mesh filename="file://$(find astribot_s1_description)/meshes/s1_torso/link4.obj"/>
+					<mesh filename="file://$(find astribot_s1_description)/meshes/s1_torso/link4.glb"/>
 				</geometry>
 			</visual>
@@ -210,5 +210,5 @@
 			<visual>
 				<geometry>
-					<mesh filename="file://$(find astribot_s1_description)/meshes/s1_head/base.obj"/>
+					<mesh filename="file://$(find astribot_s1_description)/meshes/s1_head/base.glb"/>
 				</geometry>
 			</visual>
@@ -229,5 +229,5 @@
 			<visual>
 				<geometry>
-					<mesh filename="file://$(find astribot_s1_description)/meshes/s1_head/link1.obj"/>
+					<mesh filename="file://$(find astribot_s1_description)/meshes/s1_head/link1.glb"/>
 				</geometry>
 			</visual>
@@ -249,5 +249,5 @@
 			<visual>
 				<geometry>
-					<mesh filename="file://$(find astribot_s1_description)/meshes/s1_head/link2.obj"/>
+					<mesh filename="file://$(find astribot_s1_description)/meshes/s1_head/link2.glb"/>
 				</geometry>
 			</visual>
