Commit message: Dexfoce w1 (#15)
* add dexforce w1 ros2 control

* add brainco revo2 config

* update mesh to glb for astribot s1

* agibot g1 update mesh to glb

* add zerith h1

* zerith h1 mesh cleaned

* add angellun omniwheel

* using angellun omniwheel

* remove arx and using submodules

* remove arx and using submodules

* remove Ubtech and add as submodule from robot-descriptions-ubtech

* update readme

* update readme

File: humanoid/Astribot/astribot_s1_description/xacro/components/s1_arm.xacro (robot description, xacro)
@@ -28,5 +28,5 @@
 			<visual>
 				<geometry>
-					<mesh filename="file://$(find astribot_s1_description)/meshes/s1_arm/base.obj" scale="1 ${direction} 1"/>
+					<mesh filename="file://$(find astribot_s1_description)/meshes/s1_arm/base.glb" scale="1 ${direction} 1"/>
 				</geometry>
 			</visual>
@@ -40,5 +40,5 @@
 			<visual>
 				<geometry>
-					<mesh filename="file://$(find astribot_s1_description)/meshes/s1_arm/link1.obj"/>
+					<mesh filename="file://$(find astribot_s1_description)/meshes/s1_arm/link1.glb"/>
 				</geometry>
 			</visual>
@@ -70,5 +70,5 @@
 			<visual>
 				<geometry>
-					<mesh filename="file://$(find astribot_s1_description)/meshes/s1_arm/link2.obj" scale="1 1 ${direction} "/>
+					<mesh filename="file://$(find astribot_s1_description)/meshes/s1_arm/link2.glb" scale="1 1 ${direction} "/>
 				</geometry>
 			</visual>
@@ -89,5 +89,5 @@
 			<visual>
 				<geometry>
-					<mesh filename="file://$(find astribot_s1_description)/meshes/s1_arm/link3.obj"/>
+					<mesh filename="file://$(find astribot_s1_description)/meshes/s1_arm/link3.glb"/>
 				</geometry>
 			</visual>
@@ -115,5 +115,5 @@
 			<visual>
 				<geometry>
-					<mesh filename="file://$(find astribot_s1_description)/meshes/s1_arm/link4.obj"/>
+					<mesh filename="file://$(find astribot_s1_description)/meshes/s1_arm/link4.glb"/>
 				</geometry>
 			</visual>
@@ -142,5 +142,5 @@
 			<visual>
 				<geometry>
-					<mesh filename="file://$(find astribot_s1_description)/meshes/s1_arm/link5.obj"/>
+					<mesh filename="file://$(find astribot_s1_description)/meshes/s1_arm/link5.glb"/>
 				</geometry>
 				<material name="">
@@ -170,5 +170,5 @@
 			<visual>
 				<geometry>
-					<mesh filename="file://$(find astribot_s1_description)/meshes/s1_arm/link6.obj"/>
+					<mesh filename="file://$(find astribot_s1_description)/meshes/s1_arm/link6.glb"/>
 				</geometry>
 			</visual>
@@ -189,5 +189,5 @@
 			<visual>
 				<geometry>
-					<mesh filename="file://$(find astribot_s1_description)/meshes/s1_arm/link7.obj"/>
+					<mesh filename="file://$(find astribot_s1_description)/meshes/s1_arm/link7.glb"/>
 				</geometry>
 			</visual>

File: humanoid/Astribot/astribot_s1_description/xacro/components/s1_gripper.xacro (robot description, xacro)
@@ -22,5 +22,5 @@
 			<visual>
 				<geometry>
-					<mesh filename="file://$(find astribot_s1_description)/meshes/s1_gripper/base.obj"/>
+					<mesh filename="file://$(find astribot_s1_description)/meshes/s1_gripper/base.glb"/>
 				</geometry>
 			</visual>
@@ -41,5 +41,5 @@
 			<visual>
 				<geometry>
-					<mesh filename="file://$(find astribot_s1_description)/meshes/s1_gripper/link1.obj"/>
+					<mesh filename="file://$(find astribot_s1_description)/meshes/s1_gripper/link1.glb"/>
 				</geometry>
 			</visual>
@@ -67,5 +67,5 @@
 			<visual>
 				<geometry>
-					<mesh filename="file://$(find astribot_s1_description)/meshes/s1_gripper/link2.obj"/>
+					<mesh filename="file://$(find astribot_s1_description)/meshes/s1_gripper/link2.glb"/>
 				</geometry>
 			</visual>
@@ -94,10 +94,10 @@
 			<visual>
 				<geometry>
-					<mesh filename="file://$(find astribot_s1_description)/meshes/s1_gripper/pad.obj"/>
+					<mesh filename="file://$(find astribot_s1_description)/meshes/s1_gripper/pad.glb"/>
 				</geometry>
 			</visual>
 			<collision>
 				<geometry>
-					<mesh filename="file://$(find astribot_s1_description)/meshes/s1_gripper/pad.obj"/>
+					<mesh filename="file://$(find astribot_s1_description)/meshes/s1_gripper/pad.glb"/>
 				</geometry>
 			</collision>
@@ -126,5 +126,5 @@
 			<visual>
 				<geometry>
-					<mesh filename="file://$(find astribot_s1_description)/meshes/s1_gripper/link1.obj" scale="-1 1 1"/>
+					<mesh filename="file://$(find astribot_s1_description)/meshes/s1_gripper/link1.glb" scale="-1 1 1"/>
 				</geometry>
 			</visual>
@@ -153,5 +153,5 @@
 			<visual>
 				<geometry>
-					<mesh filename="file://$(find astribot_s1_description)/meshes/s1_gripper/link2.obj" scale="-1 1 1"/>
+					<mesh filename="file://$(find astribot_s1_description)/meshes/s1_gripper/link2.glb" scale="-1 1 1"/>
 				</geometry>
 			</visual>
@@ -180,10 +180,10 @@
 			<visual>
 				<geometry>
-					<mesh filename="file://$(find astribot_s1_description)/meshes/s1_gripper/pad.obj" scale="-1 1 1"/>
+					<mesh filename="file://$(find astribot_s1_description)/meshes/s1_gripper/pad.glb" scale="-1 1 1"/>
 				</geometry>
 			</visual>
 			<collision>
 				<geometry>
-					<mesh filename="file://$(find astribot_s1_description)/meshes/s1_gripper/pad.obj" scale="-1 1 1"/>
+					<mesh filename="file://$(find astribot_s1_description)/meshes/s1_gripper/pad.glb" scale="-1 1 1"/>
 				</geometry>
 			</collision>

File: humanoid/Astribot/astribot_s1_description/xacro/robot.xacro (robot description, xacro)
@@ -47,15 +47,15 @@
 	<xacro:if value="${'$(arg type)' == 'revo2'}">
 		<xacro:include filename="$(find brainco_description)/xacro/revo2.xacro"/>
-		<xacro:BrainCoHand name="left" direction="1" fixed_joints="true"/>
-		<xacro:BrainCoHand name="right" direction="-1" fixed_joints="true"/>
+		<xacro:BrainCoHand name="left_hand" direction="1" fixed_joints="false"/>
+		<xacro:BrainCoHand name="right_hand" direction="-1" fixed_joints="false"/>
 		<joint name="left_gripper_fixed_joint" type="fixed">
 			<origin xyz="0 -0.048 0" rpy="1.5708 3.1416 0"/>
 			<parent link="left_link_7"/>
-			<child link="left_hand_base"/>
+			<child link="left_hand_hand_base"/>
 		</joint>
 		<joint name="right_gripper_fixed_joint" type="fixed">
 			<origin xyz="0 -0.048 0" rpy="1.5708 0 0"/>
 			<parent link="right_link_7"/>
-			<child link="right_hand_base"/>
+			<child link="right_hand_hand_base"/>
 		</joint>
 	</xacro:if>

File: humanoid/Astribot/astribot_s1_description/xacro/ros2_control/robot.xacro (robot description, xacro)
@@ -6,4 +6,6 @@
 <robot name="astribot_whole_body" xmlns:xacro="http://www.ros.org/wiki/xacro">
 	<!-- Include the base robot structure -->
+	<!-- Type argument will be inherited by robot.xacro -->
+	<xacro:arg name="type" default="gripper"/>
 	<xacro:include filename="$(find astribot_s1_description)/xacro/robot.xacro"/>
 	<!-- Import modular interface components -->
@@ -11,4 +13,6 @@
 	<xacro:include filename="$(find astribot_s1_description)/xacro/ros2_control/astribot_s1_arm_interfaces.xacro"/>
 	<xacro:include filename="$(find astribot_s1_description)/xacro/ros2_control/astribot_s1_gripper_interfaces.xacro"/>
+	<!-- Get type argument -->
+	<xacro:property name="type_arg" value="$(arg type)"/>
 	<!-- Unified ros2_control system -->
 	<ros2_control name="astribot_s1_unified_system" type="system">
@@ -32,7 +36,15 @@
 		<!-- 右臂接口 -->
 		<xacro:astribot_s1_arm_interfaces name="right"/>
-		<!-- 夹爪接口 -->
-		<xacro:astribot_s1_gripper_interfaces name="left"/>
-		<xacro:astribot_s1_gripper_interfaces name="right"/>
+		<!-- 夹爪接口或灵巧手接口 -->
+		<xacro:if value="${type_arg == 'gripper'}">
+			<xacro:astribot_s1_gripper_interfaces name="left"/>
+			<xacro:astribot_s1_gripper_interfaces name="right"/>
+		</xacro:if>
+		<!-- 灵巧手接口 -->
+		<xacro:if value="${type_arg == 'revo2'}">
+			<xacro:include filename="$(find brainco_description)/xacro/ros2_control/revo2.xacro"/>
+			<xacro:revo2_interfaces name="left_hand"/>
+			<xacro:revo2_interfaces name="right_hand"/>
+		</xacro:if>
 	</ros2_control>
 	<xacro:arg name="gazebo" default="false" />
